File: batteryboard-v02b/batteryboard.kicad_pcb (KiCad board)
At the start: 4 copper layers, 95.9 x 90.2 mm, 40 parts, among them J1 KEYSTONE-1042, J2 KEYSTONE-1042, J3 KEYSTONE-1042, J4 KEYSTONE-1042, J5 KEYSTONE-1042, J6 KEYSTONE-1042, J7 MOLEX 502352-0801, J8 Screw_Terminal_01x02, Q1 IRF7458, Q2 IRF7458, Q4 IRLML2803, U1 R5460N233AF, U2 DMP2040USS-13

Commit message: dont ask
Parts:
- removed C6: 10uF, Capacitor_SMD:C_0603_1608Metric
- removed R6: 200k, RN73H2BTTD2003A05, Resistor_SMD:R_1206_3216Metric
Routing:
- net /HEATER: track 3699.9 -> 3773.3 mm
- net PyCubed_AIN5: track 0.09 -> 63.1 mm, vias 0 -> 3
- net BM: track 4.24 -> 64.3 mm
- net PyCubed_HIN: track 0.40 -> 35.5 mm, vias 1 -> 2
- net PACK+: track 0.39 -> 34.3 mm, vias 12 -> 18
- net +3V3: track 1.44 -> 34.1 mm
- net PYCUBED_GND: track 70.8 -> 93.3 mm, vias 1 -> 4
- net B-: track 0.91 -> 17.3 mm
- net Net-(Q4-D): track 0.44 -> 16.2 mm
- net Net-(Q1-G): track 0.25 -> 15.2 mm
- net Net-(Q2-G): track 0.00 -> 7.77 mm
- net Net-(Q4-G): track 0.20 -> 6.82 mm
- net /VDD: track 0.03 -> 6.36 mm
- net Net-(U1-VC): track 0.00 -> 3.72 mm
- net Net-(C3-Pad1): track 0.04 -> 2.25 mm
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