File: batteryboard-v02b/batteryboard.kicad_sch (KiCad schematic)
At the start: 36 parts, among them J1 KEYSTONE-1042, J2 KEYSTONE-1042, J3 KEYSTONE-1042, J4 KEYSTONE-1042, J5 KEYSTONE-1042, J6 KEYSTONE-1042, J7 MOLEX 502352-0801, J8 Screw_Terminal_01x02, Q1 IRF7458, Q2 IRF7458, Q4 IRLML2803, U1 R5460N233AF, U2 DMP2040USS-13

Commit message: dont ask
Parts:
- removed C6: 10uF, Capacitor_SMD:C_0603_1608Metric, symbol Device:C
- removed R6: 200k, RN73H2BTTD2003A05, Resistor_SMD:R_1206_3216Metric, symbol Device:R_US
Other:
- note added: "MISSING CAP"
- note added: "MISSING RESISTOR"
